File: hardware/sband-antenna/sband-antenna.kicad_pcb (KiCad board)
At the start: 2 copper layers, 98 x 98 mm, 6 parts, among them J1 CONMCX002-SMD

Commit message: Atualizado
Parts:
- removed J1: CONMCX002-SMD, spacelab_lib:LINX_CONMCX002-SMD
- added J2: Conn_Coaxial, Connector_Coaxial:SMA_Amphenol_132134-10_Vertical, B.Cu at (87.7, 80.1)
- added Patch1: ~, SpaceLab:S-band_Patch, F.Cu at (70.2, 96.6)
- moved G*** 2.00 mm to (84.4, 114.2)
- moved H1 0.59 mm to (109.9, 35.8)
- moved H4 0.59 mm to (60.5, 35.8)
- moved H2 0.59 mm to (109.9, 127.4)
- moved H3 0.59 mm to (60.5, 127.4)
Routing:
- removed copper zone on F.Cu, net GND

Commit message: Patch and general project updates
Parts:
- removed Patch1: ~, SpaceLab:S-band_Patch
- moved J2 0.06 mm to (87.7, 80.1)
Routing:
- net ant: vias 0 -> 1
- added copper zone on F.Cu, net ant
