File: hardware/sband-antenna/sband-antenna.kicad_pcb (KiCad board)
At the start: 2 copper layers, 98 x 98 mm, 6 parts, among them J2 Conn_Coaxial

Commit message: main: Small adjustments
Parts:
- removed J2: Conn_Coaxial, Connector_Coaxial:SMA_Amphenol_132134-10_Vertical
- added J1: CONMCX002-SMD, spacelab_lib:LINX_CONMCX002-SMD, B.Cu at (105.9, 94.0)
- added U1: ~, SpaceLab:s-band-patch, F.Cu at (103.4, 95.5)
- moved G*** 29.1 mm to (103.2, 136.4)
- moved H2 22.7 mm to (127.9, 141.2)
- moved H3 22.7 mm to (78.5, 141.2)
- moved H1 22.7 mm to (127.9, 49.6)
- moved H4 22.7 mm to (78.5, 49.6)
Routing:
- net ant: vias 1 -> 0
- added copper zone on F.Cu, net GND
- removed copper zone on F.Cu, net ant
