File: hardware/sband-antenna/sband-antenna.kicad_sch (KiCad schematic)
At the start: 5 parts, among them J1 CONMCX002-SMD

Commit message: Atualizado
Parts:
- removed J1: CONMCX002-SMD, spacelab_lib:LINX_CONMCX002-SMD, symbol spacelab_lib:CONMCX002-SMD
- added J2: Conn_Coaxial, Connector_Coaxial:SMA_Amphenol_132134-10_Vertical, symbol Connector:Conn_Coaxial
- added Patch1: ~, SpaceLab:S-band_Patch, symbol S-band-antenna:Patch
Connections:
- net GND: now also J2.2 (Ext)
- net ant: now also J2.1 (In), Patch1.1 (coax)
Other:
- title: Shild -> S-band Antenna
Changed lines of the file:
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@@
 	(paper "A4")
 	(title_block
-		(title "Shild")
+		(title "S-band Antenna")
 		(date "2025-04-20")
 		(company "SpaceLab UFSC")
-		(comment 1 "Eng. Yunior Alcantara Guevara")
+		(comment 1 "Eng. Yunior Alcântara Guevara")
+		(comment 2 "Lucas Ryan Carneiro")
 	)
 	(rectangle
@@
 	)
 	(rectangle
-		(start 81.28 25.4)
+		(start 62.23 25.4)
 		(end 127 81.28)
 		(stroke
@@
 	(text "ANT"
 		(exclude_from_sim no)
-		(at 86.36 33.02 0)
+		(at 66.548 31.496 0)
 		(effects
 			(font
@@
 	)
 	(junction
+		(at 173.99 53.34)
+		(diameter 0)
+		(color 0 0 0 0)
+	)
+	(junction
 		(at 238.76 139.7)
 		(diameter 0)
@@
 	(wire
 		(pts
-			(xy 109.22 60.96) (xy 109.22 63.5)
-		)
-		(stroke
-			(width 0)
-			(type default)
-		)
-	)
-	(wire
-		(pts
-			(xy 182.88 54.61) (xy 182.88 57.15)
+			(xy 100.33 52.07) (xy 110.49 52.07)
+		)
+		(stroke
+			(width 0)
+			(type default)
+		)
+	)
+	(wire
+		(pts
+			(xy 168.91 48.26) (xy 173.99 48.26)
+		)
+		(stroke
+			(width 0)
+			(type default)
+		)
+	)
+	(wire
+		(pts
+			(xy 173.99 50.8) (xy 173.99 53.34)
 		)
 		(stroke
@@
 	(wire
 		(pts
-			(xy 114.3 48.26) (xy 109.22 48.26)
-		)
-		(stroke
-			(width 0)
-			(type default)
-		)
-	)
-	(wire
-		(pts
 			(xy 236.22 139.7) (xy 238.76 139.7)
 		)
@@
 	(wire
 		(pts
-			(xy 177.8 52.07) (xy 182.88 52.07)
+			(xy 173.99 55.88) (xy 173.99 53.34)
 		)
 		(stroke
@@
 	(global_label "ant"
 		(shape input)
-		(at 114.3 48.26 0)
+		(at 110.49 52.07 0)
 		(fields_autoplaced yes)
 		(effects
@@
 		)
 		(property "Intersheetrefs" "${INTERSHEET_REFS}"
-			(at 120.3089 48.26 0)
+			(at 116.4989 52.07 0)
 			(effects
 				(font
@@
 	(global_label "ant"
 		(shape input)
-		(at 177.8 52.07 180)
+		(at 168.91 48.26 180)
 		(fields_autoplaced yes)
 		(effects
@@
 		)
 		(property "Intersheetrefs" "${INTERSHEET_REFS}"
-			(at 171.7911 52.07 0)
+			(at 162.9011 48.26 0)
 			(effects
 				(font
@@
 		(lib_name "GND_1")
 		(lib_id "power:GND")
-		(at 182.88 57.15 0)
+		(at 173.99 55.88 0)
 		(unit 1)
 		(exclude_from_sim no)
@@
 		(fields_autoplaced yes)
 		(property "Reference" "#PWR018"
-			(at 182.88 63.5 0)
+			(at 173.99 62.23 0)
 			(effects
 				(font
@@
 		)
 		(property "Value" "GND"
-			(at 182.88 62.23 0)
+			(at 173.99 60.96 0)
 			(effects
 				(font
@@
 		)
 		(property "Footprint" ""
-			(at 182.88 57.15 0)
+			(at 173.99 55.88 0)
 			(effects
 				(font
@@
 		)
 		(property "Datasheet" ""
-			(at 182.88 57.15 0)
+			(at 173.99 55.88 0)
 			(effects
 				(font
@@
 		)
 		(property "Description" "Power symbol creates a global label with name \"GND\" , ground"
-			(at 182.88 57.15 0)
+			(at 173.99 55.88 0)
 			(effects
 				(font
@@
 	)
 	(symbol
+		(lib_id "Connector:Conn_Coaxial")
+		(at 173.99 48.26 0)
+		(unit 1)
+		(exclude_from_sim no)
+		(in_bom yes)
+		(on_board yes)
+		(dnp no)
+		(fields_autoplaced yes)
+		(property "Reference" "J2"
+			(at 177.8 47.2831 0)
+			(effects
+				(font
+					(size 1.27 1.27)
+				)
+				(justify left)
+			)
+		)
+		(property "Value" "Conn_Coaxial"
+			(at 177.8 49.8231 0)
+			(effects
+				(font
+					(size 1.27 1.27)
+				)
+				(justify left)
+			)
+		)
+		(property "Footprint" "Connector_Coaxial:SMA_Amphenol_132134-10_Vertical"
+			(at 173.99 48.26 0)
+			(effects
+				(font
+					(size 1.27 1.27)
+				)
+				(hide yes)
+			)
+		)
+		(property "Datasheet" "~"
+			(at 173.99 48.26 0)
+			(effects
+				(font
+					(size 1.27 1.27)
+				)
+				(hide yes)
+			)
+		)
+		(property "Description" "coaxial connector (BNC, SMA, SMB, SMC, Cinch/RCA, LEMO, ...)"
+			(at 173.99 48.26 0)
+			(effects
+				(font
+					(size 1.27 1.27)
+				)
+				(hide yes)
+			)
+		)
+		(pin "2"
+		)
+		(pin "1"
+		)
+		(instances
+			(project "sband-antenna"
+				(path "/e0ca2760-3043-4dcf-873b-96bc05a79e16"
+					(reference "J2")
+					(unit 1)
+				)
+			)
+		)
+	)
+	(symbol
 		(lib_id "Mechanical:MountingHole_Pad")
 		(at 241.3 134.62 0)
@@
 	)
 	(symbol
-		(lib_id "spacelab_lib:CONMCX002-SMD")
-		(at 185.42 54.61 0)
-		(mirror y)
-		(unit 1)
-		(exclude_from_sim no)
-		(in_bom yes)
-		(on_board yes)
-		(dnp no)
-		(property "Reference" "J1"
-			(at 190.5 54.8641 0)
-			(effects
-				(font
-					(size 1.27 1.27)
-				)
-				(justify right)
-			)
-		)
-		(property "Value" "CONMCX002-SMD"
-			(at 190.5 52.3241 0)
-			(effects
-				(font
-					(size 1.27 1.27)
-				)
-				(justify right)
-			)
-		)
-		(property "Footprint" "spacelab_lib:LINX_CONMCX002-SMD"
-			(at 185.42 54.61 0)
-			(effects
-				(font
-					(size 1.27 1.27)
-				)
-				(justify bottom)
-				(hide yes)
-			)
-		)
-		(property "Datasheet" ""
-			(at 185.42 54.61 0)
-			(effects
-				(font
-					(size 1.27 1.27)
-				)
-				(hide yes)
-			)
-		)
-		(property "Description" ""
-			(at 185.42 54.61 0)
-			(effects
-				(font
-					(size 1.27 1.27)
-				)
-				(hide yes)
-			)
-		)
-		(property "SnapEDA_Link" "https://www.snapeda.com/parts/CONMCX002-SMD/TE+Connectivity/view-part/?ref=snap"
-			(at 185.42 54.61 0)
-			(effects
-				(font
-					(size 1.27 1.27)
-				)
-				(justify bottom)
-				(hide yes)
-			)
-		)
-		(property "Check_prices" "https://www.snapeda.com/parts/CONMCX002-SMD/TE+Connectivity/view-part/?ref=eda"
-			(at 185.42 54.61 0)
-			(effects
-				(font
-					(size 1.27 1.27)
-				)
-				(justify bottom)
-				(hide yes)
-			)
-		)
-		(property "Package" "None"
-			(at 185.42 54.61 0)
-			(effects
-				(font
-					(size 1.27 1.27)
-				)
-				(justify bottom)
-				(hide yes)
-			)
-		)
-		(property "Price" "None"
-			(at 185.42 54.61 0)
-			(effects
-				(font
-					(size 1.27 1.27)
-				)
-				(justify bottom)
-				(hide yes)
-			)
-		)
-		(property "MF" "TE Connectivity"
-			(at 185.42 54.61 0)
-			(effects
-				(font
-					(size 1.27 1.27)
-				)
-				(justify bottom)
-				(hide yes)
-			)
-		)
-		(property "MP" "CONMCX002-SMD"
-			(at 185.42 54.61 0)
-			(effects
-				(font
-					(size 1.27 1.27)
-				)
-				(justify bottom)
-				(hide yes)
-			)
-		)
-		(property "Purchase-URL" "https://www.snapeda.com/api/url_track_click_mouser/?unipart_id=1707542&manufacturer=Linx Technologies&part_name=CONMCX002-SMD&search_term=None"
-			(at 185.42 54.61 0)
-			(effects
-				(font
-					(size 1.27 1.27)
-				)
-				(justify bottom)
-				(hide yes)
-			)
-		)
-		(property "Availability" "In Stock"
-			(at 185.42 54.61 0)
-			(effects
-				(font
-					(size 1.27 1.27)
-				)
-				(justify bottom)
-				(hide yes)
-			)
-		)
-		(property "Description_1" "MCX Jack 50 Ohm PCB Surface Mount"
-			(at 185.42 54.61 0)
-			(effects
-				(font
-					(size 1.27 1.27)
-				)
-				(justify bottom)
-				(hide yes)
-			)
-		)
-		(pin "S1"
-		)
-		(pin "1"
-		)
-		(pin "S2"
-		)
-		(instances
-			(project ""
-				(path "/e0ca2760-3043-4dcf-873b-96bc05a79e16"
-					(reference "J1")
-					(unit 1)
-				)
-			)
-		)
-	)
-	(symbol
-		(lib_name "GND_1")
-		(lib_id "power:GND")
-		(at 109.22 63.5 0)
+		(lib_id "S-band-antenna:Patch")
+		(at 50.8 64.77 0)
 		(unit 1)
 		(exclude_from_sim no)
@@
 		(dnp no)
 		(fields_autoplaced yes)
-		(property "Reference" "#PWR019"
-			(at 109.22 69.85 0)
-			(effects
-				(font
-					(size 1.27 1.27)
-				)
-				(hide yes)
-			)
-		)
-		(property "Value" "GND"
-			(at 109.22 68.58 0)
-			(effects
-				(font
-					(size 1.27 1.27)
-				)
-			)
-		)
-		(property "Footprint" ""
-			(at 109.22 63.5 0)
+		(property "Reference" "Patch1"
+			(at 104.14 51.4349 0)
+			(effects
+				(font
+					(size 1.27 1.27)
+				)
+				(justify left)
+			)
+		)
+		(property "Value" "~"
+			(at 104.14 53.34 0)
+			(effects
+				(font
+					(size 1.27 1.27)
+				)
+				(justify left)
+			)
+		)
+		(property "Footprint" "SpaceLab:S-band_Patch"
+			(at 50.8 64.77 0)
 			(effects
 				(font
@@
 		)
 		(property "Datasheet" ""
-			(at 109.22 63.5 0)
-			(effects
-				(font
-					(size 1.27 1.27)
-				)
-				(hide yes)
-			)
-		)
-		(property "Description" "Power symbol creates a global label with name \"GND\" , ground"
-			(at 109.22 63.5 0)
+			(at 50.8 64.77 0)
+			(effects
+				(font
+					(size 1.27 1.27)
+				)
+				(hide yes)
+			)
+		)
+		(property "Description" ""
+			(at 50.8 64.77 0)
 			(effects
 				(font
@@
 			(project "sband-antenna"
 				(path "/e0ca2760-3043-4dcf-873b-96bc05a79e16"
-					(reference "#PWR019")
+					(reference "Patch1")
 					(unit 1)
 				)

Commit message: main: Small adjustments
Parts:
- removed J2: Conn_Coaxial, Connector_Coaxial:SMA_Amphenol_132134-10_Vertical, symbol Connector:Conn_Coaxial
- removed Patch1: ~, SpaceLab:S-band_Patch, symbol S-band-antenna:Patch
- added J1: CONMCX002-SMD, spacelab_lib:LINX_CONMCX002-SMD, symbol spacelab_lib:CONMCX002-SMD
- added U1: ~, SpaceLab:s-band-patch, symbol S-band-antenna:Patch
Connections:
- net GND: now also J1.S1, J1.S2
- net ant: now also J1.1, U1.1 (coax)
Other:
- moved on the sheet: H1, H2, H3, H4
